File: elec/layout/default/simple-example.kicad_pcb (KiCad board)
At the start: 2 copper layers, 225.7 x 100.8 mm, 0 parts

Commit message: first commit
Parts:
- added R1: Chip Resistor - Surface Mount 10Ohms ±5% 1/16W 0402 RoHS, lib:R0402, F.Cu at (125.9, 27.5)
- added R2: Chip Resistor - Surface Mount 10Ohms ±5% 1/16W 0402 RoHS, lib:R0402, F.Cu at (129.9, 27.5)
Routing:
- net out: track 0.00 -> 2.99 mm
Changed lines of the file:
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@@
   )
   (net 0 "")
+  (net 1 "out")
+  (net 2 "gnd")
+  (net 3 "top")
+  (footprint "lib:R0402" (layer "F.Cu")
+    (at 129.9 27.5)
+    (descr "Resistor SMD 0402 (1005 Metric), square (rectangular) end terminal, IPC_7351 nominal, (Body size source: IPC-SM-782 page 72, https://www.pcb-3d.com/wordpress/wp-content/uploads/ipc-sm-782a_amendment_1_and_2.pdf), generated with kicad-footprint-generator")
+    (tags "resistor")
+    (attr smd)
+    (fp_text reference "R2" (at 0 -1.17) (layer "F.SilkS")
+        (effects (font (size 1 1) (thickness 0.15)))
+    )
+    (fp_text value "Chip Resistor - Surface Mount 10Ohms ±5% 1/16W 0402 RoHS" (at 0 1.17) (layer "F.Fab")
+        (effects (font (size 1 1) (thickness 0.15)))
+    )
+    (fp_text user "${REFERENCE}" (at 0 0) (layer "F.Fab")
+        (effects (font (size 0.26 0.26) (thickness 0.04)))
+    )
+    (fp_line (start -0.153641 -0.38) (end 0.153641 -0.38)
+      (stroke (width 0.12) (type solid)) (layer "F.SilkS"))
+    (fp_line (start -0.153641 0.38) (end 0.153641 0.38)
+      (stroke (width 0.12) (type solid)) (layer "F.SilkS"))
+    (fp_line (start -0.93 -0.47) (end 0.93 -0.47)
+      (stroke (width 0.05) (type solid)) (layer "F.CrtYd"))
+    (fp_line (start -0.93 0.47) (end -0.93 -0.47)
+      (stroke (width 0.05) (type solid)) (layer "F.CrtYd"))
+    (fp_line (start 0.93 -0.47) (end 0.93 0.47)
+      (stroke (width 0.05) (type solid)) (layer "F.CrtYd"))
+    (fp_line (start 0.93 0.47) (end -0.93 0.47)
+      (stroke (width 0.05) (type solid)) (layer "F.CrtYd"))
+    (fp_line (start -0.525 -0.27) (end 0.525 -0.27)
+      (stroke (width 0.1) (type solid)) (layer "F.Fab"))
+    (fp_line (start -0.525 0.27) (end -0.525 -0.27)
+      (stroke (width 0.1) (type solid)) (layer "F.Fab"))
+    (fp_line (start 0.525 -0.27) (end 0.525 0.27)
+      (stroke (width 0.1) (type solid)) (layer "F.Fab"))
+    (fp_line (start 0.525 0.27) (end -0.525 0.27)
+      (stroke (width 0.1) (type solid)) (layer "F.Fab"))
+    (pad "1" smd roundrect (at -0.51 0) (size 0.54 0.64) (layers "F.Cu" "F.Paste" "F.Mask") (roundrect_rratio 0.25)
+      (net 1 "out") (pintype "stereo"))
+    (pad "2" smd roundrect (at 0.51 0) (size 0.54 0.64) (layers "F.Cu" "F.Paste" "F.Mask") (roundrect_rratio 0.25)
+      (net 2 "gnd") (pintype "stereo"))
+    (model "${KICAD6_3DMODEL_DIR}/Resistor_SMD.3dshapes/R_0402_1005Metric.wrl"
+      (offset (xyz 0 0 0))
+      (scale (xyz 1 1 1))
+      (rotate (xyz 0 0 0))
+    )
+  )
+  (footprint "lib:R0402" (layer "F.Cu")
+    (at 125.89 27.5)
+    (descr "Resistor SMD 0402 (1005 Metric), square (rectangular) end terminal, IPC_7351 nominal, (Body size source: IPC-SM-782 page 72, https://www.pcb-3d.com/wordpress/wp-content/uploads/ipc-sm-782a_amendment_1_and_2.pdf), generated with kicad-footprint-generator")
+    (tags "resistor")
+    (attr smd)
+    (fp_text reference "R1" (at 0 -1.17) (layer "F.SilkS")
+        (effects (font (size 1 1) (thickness 0.15)))
+    )
+    (fp_text value "Chip Resistor - Surface Mount 10Ohms ±5% 1/16W 0402 RoHS" (at 0 1.17) (layer "F.Fab")
+        (effects (font (size 1 1) (thickness 0.15)))
+    )
+    (fp_text user "${REFERENCE}" (at 0 0) (layer "F.Fab")
+        (effects (font (size 0.26 0.26) (thickness 0.04)))
+    )
+    (fp_line (start -0.153641 -0.38) (end 0.153641 -0.38)
+      (stroke (width 0.12) (type solid)) (layer "F.SilkS"))
+    (fp_line (start -0.153641 0.38) (end 0.153641 0.38)
+      (stroke (width 0.12) (type solid)) (layer "F.SilkS"))
+    (fp_line (start -0.93 -0.47) (end 0.93 -0.47)
+      (stroke (width 0.05) (type solid)) (layer "F.CrtYd"))
+    (fp_line (start -0.93 0.47) (end -0.93 -0.47)
+      (stroke (width 0.05) (type solid)) (layer "F.CrtYd"))
+    (fp_line (start 0.93 -0.47) (end 0.93 0.47)
+      (stroke (width 0.05) (type solid)) (layer "F.CrtYd"))
+    (fp_line (start 0.93 0.47) (end -0.93 0.47)
+      (stroke (width 0.05) (type solid)) (layer "F.CrtYd"))
+    (fp_line (start -0.525 -0.27) (end 0.525 -0.27)
+      (stroke (width 0.1) (type solid)) (layer "F.Fab"))
+    (fp_line (start -0.525 0.27) (end -0.525 -0.27)
+      (stroke (width 0.1) (type solid)) (layer "F.Fab"))
+    (fp_line (start 0.525 -0.27) (end 0.525 0.27)
+      (stroke (width 0.1) (type solid)) (layer "F.Fab"))
+    (fp_line (start 0.525 0.27) (end -0.525 0.27)
+      (stroke (width 0.1) (type solid)) (layer "F.Fab"))
+    (pad "1" smd roundrect (at -0.51 0) (size 0.54 0.64) (layers "F.Cu" "F.Paste" "F.Mask") (roundrect_rratio 0.25)
+      (net 3 "top") (pintype "stereo"))
+    (pad "2" smd roundrect (at 0.51 0) (size 0.54 0.64) (layers "F.Cu" "F.Paste" "F.Mask") (roundrect_rratio 0.25)
+      (net 1 "out") (pintype "stereo"))
+    (model "${KICAD6_3DMODEL_DIR}/Resistor_SMD.3dshapes/R_0402_1005Metric.wrl"
+      (offset (xyz 0 0 0))
+      (scale (xyz 1 1 1))
+      (rotate (xyz 0 0 0))
+    )
+  )
   (gr_circle (center 225.62 81.79) (end 227.32 81.79)
     (stroke (width 0.1) (type solid)) (fill none) (layer "Edge.Cuts"))
@@
       (xy 69.100734 49.778315)
     )
-    (stroke (width 0) (type solid)) (fill none) (layer "Edge.Cuts"))
+    (stroke (width 0.1) (type solid)) (fill none) (layer "Edge.Cuts"))
   (gr_arc (start 261.62 113.79) (mid 260.448427 116.618427) (end 257.62 117.79)
     (stroke (width 0.1) (type solid)) (layer "Edge.Cuts"))
@@
     (effects (font (size 2 2) (thickness 0.1)) (justify left bottom))
   )
+  (segment (start 129.39 27.5) (end 126.4 27.5) (width 0.25) (layer "F.Cu") (net 1))
   (group "" (id 6c1ef9f7-0f34-47bb-ac1a-76df23fb396e)
     (members
